File: Hardware/ESP P113.sch (KiCad schematic (older format))
At the start: 55 parts, among them J1 L_In, J2 R_In, J3 L_Out, J4 R_Out, J5 AC_In, Q1 MJE15032, Q2 MJE15033, Q3 MJE15032, Q4 MJE15033, U1 LM4562

Commit message: Updated to V1.1
Parts:
- added F1: Fuse_Small, Fuse:Fuseholder_Cylinder-5x20mm_Schurter_0031_8201_Horizontal_Open, symbol Device:Fuse_Small
- added H5: MountingHole, MountingHole:MountingHole_3.2mm_M3_Pad_Via, symbol Mechanical:MountingHole
- J5: footprint TerminalBlock_Phoenix:TerminalBlock_Phoenix_MKDS-1,5-2_1x02_P5.00mm_Horizontal -> TerminalBlock_Phoenix:TerminalBlock_Phoenix_MKDS-1,5-2-5.08_1x02_P5.08mm_Horizontal
- L1, L2: footprint Inductor_SMD:L_Bourns_SRP1245A -> Inductor_THT:L_Radial_D12.5mm_P9.00mm_Fastron_09HCP
Connections:
- net at PS1.1 (AC/L), PS2.1 (AC/L): now also F1.2; no longer J5.1 (Pin_1)
- new net: F1.1, J5.1 (Pin_1)
Other:
- moved on the sheet: J5
Changed lines of the file:
@@
 Connection ~ 4850 3350
-Wire Wire Line
-	4950 3450 4750 3450
 Wire Wire Line
 	5900 1750 6000 1750
@@
 F 0 "L1" V 6450 3350 50  0000 C CNN
 F 1 "3u3" V 6350 3350 50  0000 C CNN
-F 2 "Inductor_SMD:L_Bourns_SRP1245A" H 6250 3350 50  0001 C CNN
+F 2 "Inductor_THT:L_Radial_D12.5mm_P9.00mm_Fastron_09HCP" H 6250 3350 50  0001 C CNN
 F 3 "~" H 6250 3350 50  0001 C CNN
 	1    6250 3350
@@
 F 0 "L2" V 6050 4150 50  0000 C CNN
 F 1 "3u3" V 6150 4150 50  0000 C CNN
-F 2 "Inductor_SMD:L_Bourns_SRP1245A" H 6250 4150 50  0001 C CNN
+F 2 "Inductor_THT:L_Radial_D12.5mm_P9.00mm_Fastron_09HCP" H 6250 4150 50  0001 C CNN
 F 3 "~" H 6250 4150 50  0001 C CNN
 	1    6250 4150
@@
 L Connector_Generic:Conn_01x02 J5
 U 1 1 60DC1978
-P 4550 3350
-F 0 "J5" H 4468 3567 50  0000 C CNN
-F 1 "AC_In" H 4468 3476 50  0000 C CNN
-F 2 "TerminalBlock_Phoenix:TerminalBlock_Phoenix_MKDS-1,5-2_1x02_P5.00mm_Horizontal" H 4550 3350 50  0001 C CNN
-F 3 "~" H 4550 3350 50  0001 C CNN
-	1    4550 3350
+P 4250 3350
+F 0 "J5" H 4168 3567 50  0000 C CNN
+F 1 "AC_In" H 4168 3476 50  0000 C CNN
+F 2 "TerminalBlock_Phoenix:TerminalBlock_Phoenix_MKDS-1,5-2-5.08_1x02_P5.08mm_Horizontal" H 4250 3350 50  0001 C CNN
+F 3 "~" H 4250 3350 50  0001 C CNN
+	1    4250 3350
 	-1   0    0    -1
 $EndComp
@@
 	1    0    0    -1
 $EndComp
+$Comp
+L Device:Fuse_Small F1
+U 1 1 60B148A5
+P 4650 3350
+F 0 "F1" H 4650 3443 50  0000 C CNN
+F 1 "Fuse_Small" H 4650 3444 50  0001 C CNN
+F 2 "Fuse:Fuseholder_Cylinder-5x20mm_Schurter_0031_8201_Horizontal_Open" H 4650 3350 50  0001 C CNN
+F 3 "~" H 4650 3350 50  0001 C CNN
+	1    4650 3350
+	1    0    0    -1
+$EndComp
+Wire Wire Line
+	4550 3350 4450 3350
+Wire Wire Line
+	4450 3450 4950 3450
+$Comp
+L Mechanical:MountingHole H5
+U 1 1 60C80349
+P 7300 4550
+F 0 "H5" H 7400 4596 50  0000 L CNN
+F 1 "MountingHole" H 7400 4505 50  0000 L CNN
+F 2 "MountingHole:MountingHole_3.2mm_M3_Pad_Via" H 7300 4550 50  0001 C CNN
+F 3 "~" H 7300 4550 50  0001 C CNN
+	1    7300 4550
+	1    0    0    -1
+$EndComp

Commit message: Updated to V1.2.
Parts:
- added D5, D6: LED, LED_THT:LED_D3.0mm, symbol Device:LED_Small
- added R17, R18: 1k, Resistor_SMD:R_1206_3216Metric_Pad1.42x1.75mm_HandSolder, symbol Device:R_Small
- C14, C15, C16, C17: value 330u -> 220u
- L1, L2: value 3u3 -> 4.7u; footprint Inductor_THT:L_Radial_D12.5mm_P9.00mm_Fastron_09HCP -> Inductor_SMD:L_Taiyo-Yuden_NR-80xx_HandSoldering
Connections:
- net +15: now also R17.1
- net -15: now also D6.1 (K)
- net Earth: now also D5.1 (K), R18.1
- new net: D5.2 (A), R17.2
- new net: D6.2 (A), R18.2
Other:
- moved on the sheet: C1, C10, C11, C12, C13, C14, C15, C16, C17, C2, C3, C4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
