File: Hardware/ESP P113.kicad_pcb (KiCad board)
At the start: 2 copper layers, 129.5 x 107.7 mm, 89 parts, among them J1 Gain_L_Ex, J2 Gain_R_Ex, J3 L_In, J4 R_In, J5 HPOut, J6 PE, J7 AC_L, J8 AC_N, J9 GND_Audio, K1 G6A-234P-ST15-US-DC24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

Commit message: Updated layout, re-added BOM.
Parts:
- removed the C17 at (54.1, 28.7)
- removed the C18 at (65.8, 28.7)
- removed L3, L4: 68u, Inductor_THT:L_Radial_D8.7mm_P5.00mm_Fastron_07HCP
- added C19: 1u, Capacitor_SMD:C_1206_3216Metric_Pad1.33x1.80mm_HandSolder, F.Cu at (104.9, 65.3)
- added C20: 1u, Capacitor_SMD:C_1206_3216Metric_Pad1.33x1.80mm_HandSolder, F.Cu at (102.4, 73.4)
- added R29: 0R33, Resistor_SMD:R_2512_6332Metric_Pad1.40x3.35mm_HandSolder, F.Cu at (53.1, 49.8)
- added R30: 0R33, Resistor_SMD:R_2512_6332Metric_Pad1.40x3.35mm_HandSolder, F.Cu at (72.9, 49.8)
- C1, C5: value 220p -> 47p
- C13, C14, C15, C16: value 220u -> 330u; footprint Capacitor_THT:CP_Radial_D10.0mm_P5.00mm -> Capacitor_THT:CP_Radial_D8.0mm_P3.50mm
- C21: footprint Capacitor_THT:C_Rect_L18.0mm_W6.0mm_P15.00mm_FKS3_FKP3 -> Capacitor_THT:C_Rect_L26.5mm_W8.5mm_P22.50mm_MKS4
- C4, C8: footprint Capacitor_SMD:C_1206_3216Metric_Pad1.33x1.80mm_HandSolder -> Capacitor_SMD:C_1210_3225Metric_Pad1.33x2.70mm_HandSolder
- F1: value 1A -> 200mA
- PS1: footprint ESP-P113-Compact:Converter_ACDC_RACx0-DK_THT -> ESP-P113:Converter_ACDC_RACx0-DK_THT
- R13, R3: value 1k1 -> 1k
- R14, R4: value 6k2 -> 5k6
- R15, R5: value 620 -> 560
- R16, R17, R6, R7: value 3k3 -> 6k8
- R18, R19, R8, R9: value 9.1 -> 10
- moved C17 60.1 mm to (56.6, 29.5), turned to 180 degrees
- moved C18 55.4 mm to (68.6, 29.5), turned to 180 degrees
- moved J8 25.5 mm to (49.3, 109.5), turned to 270 degrees
- moved C21 10.4 mm to (30.7, 42.9)
- moved J9 10.2 mm to (33.3, 38.6)
- moved D10 6.94 mm to (51.6, 31.0)
- moved C13 6.86 mm to (56.7, 43.7)
- moved D11 6.64 mm to (73.9, 31.0)
- moved C14 6.37 mm to (65.3, 43.7)
- moved L1 5.80 mm to (50.3, 41.9)
- moved L2 5.62 mm to (75.2, 41.9)
- moved C15 5.00 mm to (56.6, 35.1)
- moved C16 4.34 mm to (65.3, 35.1)
- moved PS1 3.31 mm to (63.0, 79.0)
- moved F1 3.05 mm to (21.1, 77.5)
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- renumbered C19 to C17, C20 to C18
Connections:
- C15 pad 1: Net-(C15-Pad1) -> VCC
- C16 pad 2: Net-(C16-Pad2) -> Mute_-
- L1 pad 2: Net-(C15-Pad1) -> VCC
- L2 pad 2: Net-(C16-Pad2) -> Mute_-
- PS1 pad 3: Net-(C14-Pad2) -> Net-(PS1-Pad3)
- PS1 pad 5: Net-(C13-Pad1) -> Net-(PS1-Pad5)
Routing:
- net Net-(J8-Pad1): track 59.6 -> 34.2 mm
- net Net-(C14-Pad2): track 0.00 -> 13.6 mm
- net Net-(C13-Pad1): track 0.00 -> 13.5 mm
- net Net-(PS1-Pad5): track 0.00 -> 7.51 mm
- net Net-(PS1-Pad3): track 0.00 -> 7.51 mm
- net VCC: track 247.9 -> 254.0 mm
- net Mute_-: track 274.9 -> 271.3 mm
- net GNDPWR: track 9.64 -> 12.2 mm
- net Net-(F1-Pad1): track 13.1 -> 14.4 mm
- added copper zone on B.Cu, net GND
- removed copper zone on B.Cu, net Mute_-
- removed copper zone on B.Cu, net Net-(C13-Pad1)
- removed copper zone on B.Cu, net Net-(C14-Pad2)
- removed copper zone on B.Cu, net Net-(C15-Pad1)
- removed copper zone on B.Cu, net Net-(C16-Pad2)
- removed copper zone on B.Cu, net VCC
Other:
- outline, holes or cut-outs redrawn
- board text added: "AC L"
- board text added: "AC N"
- board text removed: "AC In"
- board text removed: "N"

Commit message: Added RFI filter.
Parts:
- added C22: 220p, Capacitor_SMD:C_1206_3216Metric_Pad1.33x1.80mm_HandSolder, F.Cu at (118.4, 83.8)
- added C23: 220p, Capacitor_SMD:C_1206_3216Metric_Pad1.33x1.80mm_HandSolder, F.Cu at (115.8, 47.2)
- added R31: 2k2, Resistor_SMD:R_1206_3216Metric_Pad1.30x1.75mm_HandSolder, F.Cu at (118.4, 78.7)
- added R32: 2k2, Resistor_SMD:R_1206_3216Metric_Pad1.30x1.75mm_HandSolder, F.Cu at (118.4, 47.2)
- moved R1 2.54 mm to (115.8, 83.8)
- moved R5 2.54 mm to (110.7, 83.8)
- moved R3 2.54 mm to (113.3, 83.8)
- moved R4 2.54 mm to (108.2, 83.8)
Connections:
- R1 pad 1: L_In -> Net-(C22-Pad2)
- R11 pad 1: R_In -> Net-(C23-Pad2)
- R12 pad 2: R_In -> Net-(C23-Pad2)
- R2 pad 2: L_In -> Net-(C22-Pad2)
Routing:
- net Net-(C22-Pad2): track 0.00 -> 6.53 mm
- net Net-(C23-Pad2): track 0.00 -> 6.49 mm
- net L_In: track 63.6 -> 58.1 mm
- net R_In: track 26.7 -> 22.1 mm
- net L_Out: track 115.6 -> 113.0 mm
- net Net-(J1-Pad2): track 22.8 -> 21.8 mm
