File: Amp and PSU/Hardware/ESP P113.kicad_pcb (KiCad board)
At the start: 2 copper layers, 100.3 x 72.4 mm, 61 parts, among them J1 L_In, J2 R_In, J3 L_Out, J4 R_Out, J5 AC_In, Q1 MJE15032, Q2 MJE15033, Q3 MJE15032, Q4 MJE15033, U1 LM4562

Commit message: Added version with no PSU
Other:
- board text added: "ESP P113 Layout by Aria V1.2"
- board text removed: "ESP P113 Layout by Aria V1.1"
