File: Amp_PSU/Hardware/ESP P113.sch (KiCad schematic (older format))
At the start: 61 parts, among them J1 L_In, J2 R_In, J3 L_Out, J4 R_Out, J5 AC_In, Q1 MJE15032, Q2 MJE15033, Q3 MJE15032, Q4 MJE15033, U1 LM4562

Commit message: Changed output resistors to THT 0.5W versions. Removed amp-only version. Added disclaimer on board.
Parts:
- R15, R16, R7, R8: footprint Resistor_SMD:R_1206_3216Metric_Pad1.42x1.75mm_HandSolder -> Resistor_THT:R_Axial_DIN0207_L6.3mm_D2.5mm_P7.62mm_Horizontal
Connections:
- net at F1.1: now also J5.2 (Pin_2); no longer J5.1 (Pin_1)
- net at PS1.2 (AC/N), PS2.2 (AC/N): now also J5.1 (Pin_1); no longer J5.2 (Pin_2)

Commit message: Updated to V2.0.
Parts:
- removed C14, C15, C16: 220u, Capacitor_THT:CP_Radial_D8.0mm_P3.50mm, symbol Device:CP_Small
- removed C4, C8: 100u, Capacitor_THT:CP_Radial_D6.3mm_P2.50mm, symbol Device:CP_Small
- removed F1: Fuse_Small, Fuse:Fuseholder_Cylinder-5x20mm_Schurter_0031_8201_Horizontal_Open, symbol Device:Fuse_Small
- removed H1: Star_Ground, MountingHole:MountingHole_3.2mm_M3_Pad_Via, symbol Mechanical:MountingHole_Pad
- added C11, C4: 22pF, Capacitor_SMD:C_0805_2012Metric_Pad1.15x1.40mm_HandSolder, symbol Device:C_Small
- added C13, C6: 100u, Capacitor_THT:CP_Radial_D6.3mm_P2.50mm, symbol Device:CP_Small
- added C14, C15, C7: 100n, Capacitor_SMD:C_0805_2012Metric_Pad1.15x1.40mm_HandSolder, symbol Device:C_Small
- added C2: 220p, Capacitor_SMD:C_0805_2012Metric_Pad1.15x1.40mm_HandSolder, symbol Device:C_Small
- added C20, C21: 1u, Capacitor_SMD:C_0805_2012Metric_Pad1.15x1.40mm_HandSolder, symbol Device:C_Small
- added C22, C23: 10u, Capacitor_THT:CP_Radial_D6.3mm_P2.50mm, symbol Device:CP_Small
- added C24: 220u, Capacitor_THT:CP_Radial_D8.0mm_P3.50mm, symbol Device:CP_Small
- added C26: 10nF, Capacitor_THT:C_Disc_D16.0mm_W5.0mm_P10.00mm, symbol Device:C_Small
- added D7, D8: TVS, Diode_SMD:D_SMB, symbol Device:D_Zener_Small
- added H5: MountingHole_Pad, MountingHole:MountingHole_3.2mm_M3_Pad_Via, symbol Mechanical:MountingHole_Pad
- added J6: Gain_L_Ex, Connector_JST:JST_XH_B2B-XH-A_1x02_P2.50mm_Vertical, symbol Connector_Generic:Conn_01x02
- added J7: Gain_R_Ex, Connector_JST:JST_XH_B2B-XH-A_1x02_P2.50mm_Vertical, symbol Connector_Generic:Conn_01x02
- added R1, R12: 470, Resistor_SMD:R_1206_3216Metric_Pad1.42x1.75mm_HandSolder, symbol Device:R_Small
- added R11, R22: 10, Resistor_SMD:R_1206_3216Metric_Pad1.42x1.75mm_HandSolder, symbol Device:R_Small
- added R17, R6: 9k1, Resistor_SMD:R_1206_3216Metric_Pad1.42x1.75mm_HandSolder, symbol Device:R_Small
- added R25, R26: 3, Resistor_THT:R_Axial_DIN0614_L14.3mm_D5.7mm_P15.24mm_Horizontal, symbol Device:R_Small
- added RV1, RV2: MOV, Capacitor_THT:C_Disc_D14.5mm_W5.0mm_P7.50mm, symbol Custom_Parts:Varistor_Small
- added SW1: Gain_L, Button_Switch_THT:SW_DIP_SPSTx01_Slide_6.7x4.1mm_W7.62mm_P2.54mm_LowProfile, symbol Switch:SW_SPST
- added SW2: Gain_R, Button_Switch_THT:SW_DIP_SPSTx01_Slide_6.7x4.1mm_W7.62mm_P2.54mm_LowProfile, symbol Switch:SW_SPST
- C9: value 100n -> 220p
- J5: footprint TerminalBlock_Phoenix:TerminalBlock_Phoenix_MKDS-1,5-2-5.08_1x02_P5.08mm_Horizontal -> TerminalBlock_Phoenix:TerminalBlock_Phoenix_MKDS-1,5-3-5.08_1x03_P5.08mm_Horizontal; symbol Connector_Generic:Conn_01x02 -> Connector_Generic:Conn_01x03
- PS1, PS2: symbol Converter_ACDC:IRM-20-15 -> Converter_ACDC:IRM-20-24
- Q1, Q3: value MJE15032 -> BD139; footprint Package_TO_SOT_THT:TO-220-3_Vertical -> Package_TO_SOT_THT:TO-126-3_Vertical; symbol Device:Q_PNP_BCE -> Transistor_BJT:BD139
- Q2, Q4: value MJE15033 -> BD140; footprint Package_TO_SOT_THT:TO-220-3_Vertical -> Package_TO_SOT_THT:TO-126-3_Vertical; symbol Device:Q_PNP_BCE -> Transistor_BJT:BD140
- R14: renamed from R10; value 1k -> 470
- R16: renamed from R12; value 3k3 -> 5k1
- R3: renamed from R2; value 1k -> 470
- R5: renamed from R4; value 3k3 -> 5k1
- U1: value LM4562 -> OPA1642
- renumbered C6 to C10, C7 to C12, C10 to C16, C11 to C17, C12 to C18, C13 to C19, C17 to C25, C2 to C3, C3 to C5, C5 to C8, H5 to H1, R8 to R10, R9 to R13, R11 to R15, R13 to R18, R14 to R19, R1 to R2, R15 to R20, R16 to R21, R17 to R23, R18 to R24, R3 to R4, R5 to R7, R6 to R8, R7 to R9
Connections:
- net +15: now also C15.2, C24.1; no longer C9.2
- net -15: now also Q2.2 (C), Q4.2 (C), C15.1; no longer C9.1, Q2.3 (E), Q4.3 (E)
- net L_Out: now also J6.1 (Pin_1), R11.2, R6.2, SW1.2 (B); no longer R5.2
- net R_Out: now also J7.1 (Pin_1), R17.2, R22.2, SW2.2 (B); no longer R16.2
- net at R2.1, R3.2: now also R1.1; no longer C1.1
- net at C3.1, R5.1, U1.2 (-): now also C4.2, R6.1
- net at C5.1, D1.2 (A), R7.2: now also Q1.3 (B); no longer Q1.1 (B)
- net at C5.2, D1.1 (K), D2.2 (A)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: now also C4.1, C6.1
- net at D2.1 (K), R8.1: now also Q2.3 (B), C6.2; no longer Q2.1 (B)
- net at R9.1: now also Q1.1 (E); no longer Q1.3 (E)
- net at R10.2: now also Q2.1 (E); no longer Q2.2 (C)
- net GNDREF: now reaches J5.2 (Pin_2)
- net GNDREF: now also C26.1
- net at PS1.1 (AC/L): now also R25.1; no longer PS2.1 (AC/L)
- net at J5.1 (Pin_1), PS1.2 (AC/N), PS2.2 (AC/N): now also RV1.2, RV2.2
- net at R13.1, R14.2: now also R12.1; no longer C8.1
- net at C10.1, R16.1, U1.6 (-): now also C11.2, R17.1
- net at C12.1, D3.2 (A), R18.2: now also Q3.3 (B); no longer Q3.1 (B)
- net at C12.2, D3.1 (K), D4.2 (A)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: now also C11.1, C13.1
- net at D4.1 (K), R19.1: now also Q4.3 (B), C13.2; no longer Q4.1 (B)
- net at R20.1: now also Q3.1 (E); no longer Q3.3 (E)
- net at R21.2: now also Q4.1 (E); no longer Q4.2 (C)
- net at L1.1, PS1.4 (+Vo): now also C20.1, C22.1, D7.1 (K)
- net at L2.1, PS2.3 (-Vo): now also C21.2, C23.2, D8.2 (A)
- net Earth renamed GND
- net GND: now also C9.1, C14.1, C2.1, C20.2, C21.1, C22.2, C23.1, C24.2, C26.2, C7.1, D7.2 (A), D8.1 (K), H5.1
- new net: C1.1, C2.2, R1.2
- new net: J6.2 (Pin_2), R5.2, SW1.1 (A)
- new net: J5.3 (Pin_3), R25.2, R26.2, RV1.1, RV2.1
- new net: PS2.1 (AC/L), R26.1
- new net: C7.2, R11.1
- new net: C14.2, R22.1
- new net: C8.1, C9.2, R12.2
- new net: J7.2 (Pin_2), R16.2, SW2.1 (A)
Other:
- moved on the sheet: C1, C10, C12, C16, C17, C18, C19, C25, C3, C5, C8, D1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

Commit message: Changed layout
Parts:
- removed C26: 10nF, Capacitor_THT:C_Disc_D16.0mm_W5.0mm_P10.00mm, symbol Device:C_Small
- removed H5: MountingHole_Pad, MountingHole:MountingHole_3.2mm_M3_Pad_Via, symbol Mechanical:MountingHole_Pad
- removed J5: AC_In, TerminalBlock_Phoenix:TerminalBlock_Phoenix_MKDS-1,5-3-5.08_1x03_P5.08mm_Horizontal, symbol Connector_Generic:Conn_01x03
- added J7: AC_In, TerminalBlock_Phoenix:TerminalBlock_Phoenix_MKDS-1,5-2-5.08_1x02_P5.08mm_Horizontal, symbol Connector_Generic:Conn_01x02
- renumbered J6 to J5, J7 to J6
Connections:
- net at R25.2, R26.2, RV1.1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: now also J7.1 (Pin_1)
- net at PS1.2 (AC/N), PS2.2 (AC/N), RV1.2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: now also J7.2 (Pin_2)
Changed lines of the file:
@@
 $EndComp
-$Comp
-L Connector_Generic:Conn_01x03 J5
-U 1 1 60DC1978
-P 4450 3750
-F 0 "J5" H 4400 4050 50  0000 C CNN
-F 1 "AC_In" H 4400 3950 50  0000 C CNN
-F 2 "TerminalBlock_Phoenix:TerminalBlock_Phoenix_MKDS-1,5-3-5.08_1x03_P5.08mm_Horizontal" H 4450 3750 50  0001 C CNN
-F 3 "~" H 4450 3750 50  0001 C CNN
-	1    4450 3750
-	-1   0    0    1
-$EndComp
-Wire Wire Line
-	4750 3750 4650 3750
 $Comp
 L Mechanical:MountingHole H2
@@
 F 3 "~" H 9700 3700 50  0001 C CNN
 	1    9700 3700
-	1    0    0    -1
-$EndComp
-$Comp
-L power:GNDREF #PWR09
-U 1 1 60C8A29C
-P 4750 3950
-F 0 "#PWR09" H 4750 3700 50  0001 C CNN
-F 1 "GNDREF" H 4755 3777 50  0000 C CNN
-F 2 "" H 4750 3950 50  0001 C CNN
-F 3 "" H 4750 3950 50  0001 C CNN
-	1    4750 3950
 	1    0    0    -1
 $EndComp
@@
 Wire Wire Line
 	5050 4250 5050 3650
-Connection ~ 5050 3650
-Connection ~ 4950 3850
-$Comp
-L Mechanical:MountingHole_Pad H5
-U 1 1 6105B2FD
-P 9650 4500
-F 0 "H5" V 9604 4650 50  0000 L CNN
-F 1 "MountingHole_Pad" V 9695 4650 50  0000 L CNN
-F 2 "MountingHole:MountingHole_3.2mm_M3_Pad_Via" H 9650 4500 50  0001 C CNN
-F 3 "~" H 9650 4500 50  0001 C CNN
-	1    9650 4500
-	0    1    1    0
-$EndComp
-$Comp
-L power:GNDPWR #PWR0101
-U 1 1 6105CB6D
-P 9550 4500
-F 0 "#PWR0101" H 9550 4300 50  0001 C CNN
-F 1 "GNDPWR" H 9554 4346 50  0000 C CNN
-F 2 "" H 9550 4450 50  0001 C CNN
-F 3 "" H 9550 4450 50  0001 C CNN
-	1    9550 4500
-	1    0    0    -1
-$EndComp
 $Comp
 L Converter_ACDC:IRM-20-24 PS1
@@
 	0    1    1    0
 $EndComp
-$Comp
-L Device:C_Small C26
-U 1 1 60D41E0A
-P 8650 4050
-F 0 "C26" V 8421 4050 50  0000 C CNN
-F 1 "10nF" V 8512 4050 50  0000 C CNN
-F 2 "Capacitor_THT:C_Disc_D16.0mm_W5.0mm_P10.00mm" H 8650 4050 50  0001 C CNN
-F 3 "~" H 8650 4050 50  0001 C CNN
-	1    8650 4050
-	0    1    1    0
-$EndComp
 Text GLabel 7750 4450 2    50   Input ~ 0
 -15
-Connection ~ 8450 4050
-Wire Wire Line
-	8450 4050 8550 4050
-$Comp
-L power:GNDREF #PWR012
-U 1 1 60D474EF
-P 8850 4150
-F 0 "#PWR012" H 8850 3900 50  0001 C CNN
-F 1 "GNDREF" H 8855 3977 50  0000 C CNN
-F 2 "" H 8850 4150 50  0001 C CNN
-F 3 "" H 8850 4150 50  0001 C CNN
-	1    8850 4150
-	1    0    0    -1
-$EndComp
-Wire Wire Line
-	8450 4050 8450 4150
-Wire Wire Line
-	8850 4150 8850 4050
-Wire Wire Line
-	8850 4050 8750 4050
 $Comp
 L Converter_ACDC:IRM-20-24 PS2
@@
 	6450 4050 6450 3950
 Wire Wire Line
-	8050 4050 8450 4050
+	8050 4050 8350 4050
 Connection ~ 8050 4050
 $Comp
@@
 L power:GNDPWR #PWR011
 U 1 1 60C88A62
-P 8450 4150
-F 0 "#PWR011" H 8450 3950 50  0001 C CNN
-F 1 "GNDPWR" H 8454 3996 50  0000 C CNN
-F 2 "" H 8450 4100 50  0001 C CNN
-F 3 "" H 8450 4100 50  0001 C CNN
-	1    8450 4150
-	1    0    0    -1
-$EndComp
-Wire Wire Line
-	4750 3750 4750 3950
+P 8350 4150
+F 0 "#PWR011" H 8350 3950 50  0001 C CNN
+F 1 "GNDPWR" H 8354 3996 50  0000 C CNN
+F 2 "" H 8350 4100 50  0001 C CNN
+F 3 "" H 8350 4100 50  0001 C CNN
+	1    8350 4150
+	1    0    0    -1
+$EndComp
 Wire Wire Line
 	4950 4450 5150 4450
@@
 	5050 4250 5150 4250
 Wire Wire Line
-	5050 3650 5150 3650
-Wire Wire Line
 	4950 3850 5150 3850
-Wire Wire Line
-	4650 3650 5050 3650
-Wire Wire Line
-	4650 3850 4950 3850
-Wire Wire Line
-	4950 3850 4950 4450
 $Comp
 L Switch:SW_SPST SW1
@@
 $EndComp
 $Comp
-L Connector_Generic:Conn_01x02 J7
+L Connector_Generic:Conn_01x02 J6
 U 1 1 612DBFA6
 P 7750 3200
-F 0 "J7" V 7622 3280 50  0000 L CNN
+F 0 "J6" V 7622 3280 50  0000 L CNN
 F 1 "Gain_R_Ex" V 7713 3280 50  0000 L CNN
 F 2 "Connector_JST:JST_XH_B2B-XH-A_1x02_P2.50mm_Vertical" H 7750 3200 50  0001 C CNN
@@
 	3350 2800 3350 2900
 $Comp
-L Connector_Generic:Conn_01x02 J6
+L Connector_Generic:Conn_01x02 J5
 U 1 1 6135A97B
 P 3200 3200
-F 0 "J6" V 3072 3280 50  0000 L CNN
+F 0 "J5" V 3072 3280 50  0000 L CNN
 F 1 "Gain_L_Ex" V 3163 3280 50  0000 L CNN
 F 2 "Connector_JST:JST_XH_B2B-XH-A_1x02_P2.50mm_Vertical" H 3200 3200 50  0001 C CNN
@@
 	2950 3000 2950 2900
 Connection ~ 2950 2900
+Wire Wire Line
+	8350 4150 8350 4050
+Wire Wire Line
+	4950 3650 5050 3650
+Connection ~ 5050 3650
+Wire Wire Line
+	5050 3650 5150 3650
+Wire Wire Line
+	4950 3850 4950 4450
+$Comp
+L Connector_Generic:Conn_01x02 J7
+U 1 1 60D33A75
+P 4750 3650
+F 0 "J7" H 4668 3867 50  0000 C CNN
+F 1 "AC_In" H 4668 3776 50  0000 C CNN
+F 2 "TerminalBlock_Phoenix:TerminalBlock_Phoenix_MKDS-1,5-2-5.08_1x02_P5.08mm_Horizontal" H 4750 3650 50  0001 C CNN
+F 3 "~" H 4750 3650 50  0001 C CNN
+	1    4750 3650
+	-1   0    0    -1
+$EndComp
+Wire Wire Line
+	4950 3750 4950 3850
+Connection ~ 4950 3850
 $EndSCHEMATC

Commit message: Minor correction
Parts:
- J7: footprint TerminalBlock_Phoenix:TerminalBlock_Phoenix_MKDS-1,5-2-5.08_1x02_P5.08mm_Horizontal -> MountingHole:MountingHole_3.2mm_M3_Pad_Via
Changed lines of the file:
@@
 F 0 "J7" H 4668 3867 50  0000 C CNN
 F 1 "AC_In" H 4668 3776 50  0000 C CNN
-F 2 "TerminalBlock_Phoenix:TerminalBlock_Phoenix_MKDS-1,5-2-5.08_1x02_P5.08mm_Horizontal" H 4750 3650 50  0001 C CNN
+F 2 "MountingHole:MountingHole_3.2mm_M3_Pad_Via" H 4750 3650 50  0001 C CNN
 F 3 "~" H 4750 3650 50  0001 C CNN
 	1    4750 3650
